File: mega_shield3.brd (EAGLE design)
At the start: 103.8 x 58.7 mm, 36 parts, among them IC1 L298, IC2 LM2937ET-5V, J2 Mega R3

Commit message: final gerber files
Parts:
- added C5, C6, C7, C8, C9: 0.1 uF, rcl:C025-050X050
- moved C4 13.2 mm to (57.4, 22.1), turned to 180 degrees
- moved D7 1.76 mm to (25.9, 39.9)
- moved LED2 1.76 mm to (51.3, 25.4)
- moved R3 1.76 mm to (51.3, 15.5)
- moved LED5 1.76 mm to (5.11, 49.8)
- moved BNO055 1.76 mm to (88.9, 46.8)
- moved C3 1.76 mm to (85.4, 42.2)
- moved D1 1.76 mm to (42.2, 39.9)
- moved LED1 1.76 mm to (51.3, 32.3)
- moved R5 1.76 mm to (72.2, 35.6)
- moved R6 1.76 mm to (67.6, 35.6)
- moved R7 1.76 mm to (80.8, 35.6)
- moved R2 1.76 mm to (25.4, 12.0)
- moved C1 1.76 mm to (12.5, 9.17)
- moved C2 1.76 mm to (3.58, 15.8)
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Connections:
- new net N$1: C5.1, MPR121.1
- new net N$2: C6.1, MPR121.3
- new net N$5: C7.1, MPR121.5
- new net N$6: C8.1, MPR121.7
- new net N$8: C9.1, MPR121.9
- net GND: now also C5.2, C6.2, C7.2, C8.2, C9.2
Routing:
- net N$8: track 0.00 -> 6.49 mm
- net N$1: track 0.00 -> 6.28 mm
- net N$6: track 0.00 -> 5.97 mm
- net N$2: track 0.00 -> 5.75 mm
- net N$5: track 0.00 -> 5.44 mm
- net MEGASCL: track 45.0 -> 43.8 mm
- net MEGA_5V: track 177.6 -> 176.9 mm, vias 0 -> 1
- net N$7: track 13.2 -> 12.6 mm
Other:
- board size 103.8 x 58.7 mm -> 101.6 x 53.3 mm
- board text added: "Carnegie Malones"
- board text removed: "CARNEGIE MALONES"
