File: mega_shield3.sch (EAGLE design)
At the start: 36 parts, among them IC1 L298, IC2 LM2937ET-5V, J2 Mega R3

Commit message: final gerber files
Parts:
- added C5, C6, C7, C8, C9: 0.1 uF, rcl:C-US025-050X050
Connections:
- new net N$1: C5.1, MPR121.1
- new net N$2: C6.1, MPR121.3
- new net N$5: C7.1, MPR121.5
- new net N$6: C8.1, MPR121.7
- new net N$8: C9.1, MPR121.9
- net GND: now also C5.2, C6.2, C7.2, C8.2, C9.2
Changed lines of the file:
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@@
 <part name="GND15" library="supply1" deviceset="GND" device=""/>
 <part name="SLIDE_SW" library="arduinoShield" deviceset="E-SWITCH_500SSP1S2M2QEA" device=""/>
+<part name="C5" library="rcl" deviceset="C-US" device="025-050X050" value="0.1 uF"/>
+<part name="GND16" library="supply1" deviceset="GND" device=""/>
+<part name="C6" library="rcl" deviceset="C-US" device="025-050X050" value="0.1 uF"/>
+<part name="GND17" library="supply1" deviceset="GND" device=""/>
+<part name="C7" library="rcl" deviceset="C-US" device="025-050X050" value="0.1 uF"/>
+<part name="GND18" library="supply1" deviceset="GND" device=""/>
+<part name="C8" library="rcl" deviceset="C-US" device="025-050X050" value="0.1 uF"/>
+<part name="GND19" library="supply1" deviceset="GND" device=""/>
+<part name="C9" library="rcl" deviceset="C-US" device="025-050X050" value="0.1 uF"/>
+<part name="GND21" library="supply1" deviceset="GND" device=""/>
 </parts>
 <sheets>
@@
 <instance part="GND15" gate="1" x="71.12" y="-142.24"/>
 <instance part="SLIDE_SW" gate="G$1" x="1.778" y="-46.482" rot="R90"/>
+<instance part="C5" gate="G$1" x="-48.26" y="17.78" rot="R270"/>
+<instance part="GND16" gate="1" x="-53.34" y="15.24"/>
+<instance part="C6" gate="G$1" x="-48.26" y="10.16" rot="R270"/>
+<instance part="GND17" gate="1" x="-53.34" y="7.62"/>
+<instance part="C7" gate="G$1" x="-48.26" y="2.54" rot="R270"/>
+<instance part="GND18" gate="1" x="-53.34" y="0"/>
+<instance part="C8" gate="G$1" x="-48.26" y="-5.08" rot="R270"/>
+<instance part="GND19" gate="1" x="-53.34" y="-7.62"/>
+<instance part="C9" gate="G$1" x="-48.26" y="-12.7" rot="R270"/>
+<instance part="GND21" gate="1" x="-53.34" y="-15.24"/>
 </instances>
 <busses>
@@
 <wire x1="50.8" y1="-139.7" x2="71.12" y2="-139.7" width="0.1524" layer="91"/>
 </segment>
+<segment>
+<pinref part="C5" gate="G$1" pin="2"/>
+<pinref part="GND16" gate="1" pin="GND"/>
+</segment>
+<segment>
+<pinref part="C6" gate="G$1" pin="2"/>
+<pinref part="GND17" gate="1" pin="GND"/>
+</segment>
+<segment>
+<pinref part="C7" gate="G$1" pin="2"/>
+<pinref part="GND18" gate="1" pin="GND"/>
+</segment>
+<segment>
+<pinref part="C8" gate="G$1" pin="2"/>
+<pinref part="GND19" gate="1" pin="GND"/>
+</segment>
+<segment>
+<pinref part="C9" gate="G$1" pin="2"/>
+<pinref part="GND21" gate="1" pin="GND"/>
+</segment>
 </net>
 <net name="MEGASDA" class="0">
@@
 </segment>
 </net>
+<net name="N$1" class="0">
+<segment>
+<pinref part="MPR121" gate="G$1" pin="1"/>
+<pinref part="C5" gate="G$1" pin="1"/>
+</segment>
+</net>
+<net name="N$2" class="0">
+<segment>
+<pinref part="MPR121" gate="G$1" pin="3"/>
+<pinref part="C6" gate="G$1" pin="1"/>
+</segment>
+</net>
+<net name="N$5" class="0">
+<segment>
+<pinref part="MPR121" gate="G$1" pin="5"/>
+<pinref part="C7" gate="G$1" pin="1"/>
+</segment>
+</net>
+<net name="N$6" class="0">
+<segment>
+<pinref part="MPR121" gate="G$1" pin="7"/>
+<pinref part="C8" gate="G$1" pin="1"/>
+</segment>
+</net>
+<net name="N$8" class="0">
+<segment>
+<pinref part="MPR121" gate="G$1" pin="9"/>
+<pinref part="C9" gate="G$1" pin="1"/>
+</segment>
+</net>
