File: mega_shield_despair.brd (EAGLE design)
At the start: 101.6 x 53.3 mm, 41 parts, among them IC1 L298, IC2 LM2937ET-5V, J2 Mega R3

Commit message: add despair version
Parts:
- removed LED1, LED3: GREEN, adafruit:LED3MM
- removed LED2, LED4: RED, adafruit:LED3MM
- removed R3, R4: 2.2K, rcl:0207/10
- moved R5 5.31 mm to (66.9, 35.6)
- moved R6 4.37 mm to (72.0, 35.6)
- moved SLIDE_SW 2.39 mm to (7.37, 21.6)
- moved D1 1.24 mm to (43.4, 39.9)
- moved D2 1.24 mm to (43.4, 44.2)
- moved C3 0.35 mm to (85.6, 42.0)
- moved R9 0.10 mm to (5.11, 41.3)
Connections:
- removed net N$12: LED3.K, LED4.K, R4.2
- removed net N$7: LED1.K, LED2.K, R3.2
- net GND: no longer R3.1, R4.1
- net MOT1: no longer LED2.A
- net MOT2: no longer LED1.A
- net MOT3: no longer LED4.A
- net MOT4: no longer LED3.A
Routing:
- net MEGASCL: track 43.8 -> 77.6 mm
- net MEGASDA: track 36.7 -> 64.8 mm
- net MOT1: track 49.6 -> 33.1 mm, vias 2 -> 0
- net N$7: track 12.6 -> 0.00 mm
- net N$12: track 12.2 -> 0.00 mm
- net GND: track 0.00 -> 8.52 mm
- net MOT3: track 42.1 -> 37.6 mm
- net MEGA3: track 19.0 -> 22.7 mm
- net MEGA_5V: track 176.9 -> 174.2 mm, vias 1 -> 0
- net MOT4: track 53.2 -> 50.8 mm
- net MEGA42: track 83.3 -> 81.1 mm
- net LDO_5V: track 60.7 -> 61.9 mm
- net 12V_RAIL: track 69.7 -> 68.6 mm
- net MEGA6: track 33.8 -> 34.5 mm
- net MOT2: track 49.9 -> 49.2 mm
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Other:
- board text added: "Por que no los dos?"
- board text added: "We'll carry on"
- board text added: "Welcome to the Black Parade"
